Commit message: update direction of motor

File: tracked_description/urdf/gazebo/tracked_arm_continuous_position.xacro (robot description, xacro)
@@ -69,5 +69,5 @@
     <child link="link3"/>
     <origin xyz="0 0 ${height2}" rpy="0 0 0"/>
-    <axis xyz="0 1 0"/>
+    <axis xyz="0 -1 0"/>
 <!--    <limit lower="${-PI}" upper="${PI}" effort="1" velocity="1" />-->
     <dynamics damping="0.7"/>

File: tracked_description/urdf/gazebo/tracked_arm_revolute_effort.xacro (robot description, xacro)
@@ -69,5 +69,5 @@
     <child link="link3"/>
     <origin xyz="0 0 ${height2}" rpy="0 0 0"/>
-    <axis xyz="0 1 0"/>
+    <axis xyz="0 -1 0"/>
     <limit lower="${-PI}" upper="${PI}" effort="1000000" velocity="1" />
     <dynamics damping="0.7"/>

File: tracked_description/urdf/rviz/tracked_arm_continuous_position_rviz.xacro (robot description, xacro)
@@ -69,5 +69,5 @@
     <child link="link3"/>
     <origin xyz="0 0 ${height2}" rpy="0 0 0"/>
-    <axis xyz="0 1 0"/>
+    <axis xyz="0 -1 0"/>
 <!--    <limit lower="${-PI}" upper="${PI}" effort="1" velocity="1" />-->
     <dynamics damping="0.7"/>
