Commit message: update arm motor velocity

File: tracked_description/urdf/gazebo/tracked_arm_revolute_position.xacro (robot description, xacro)
@@ -7,5 +7,5 @@
     <origin xyz="0 0 ${l_bh/2}" rpy="0 0 ${PI}"/>
     <axis xyz="0 0 1"/>
-    <limit lower="${-PI}" upper="${PI}" effort="10" velocity="1" />
+    <limit lower="${-PI}" upper="${PI}" effort="10" velocity="3" />
     <dynamics damping="0.7"/>
   </joint>
@@ -38,5 +38,5 @@
     <origin xyz="0 0 ${m_h}" rpy="0 0 0"/>
     <axis xyz="0 -1 0"/>
-    <limit lower="${-PI}" upper="${PI}" effort="1000000" velocity="1" />
+    <limit lower="${-PI}" upper="${PI}" effort="1000000" velocity="3" />
     <dynamics damping="0.7"/>
   </joint>
@@ -70,5 +70,5 @@
     <origin xyz="0 0 ${height2}" rpy="0 0 0"/>
     <axis xyz="0 1 0"/>
-    <limit lower="${-PI}" upper="${PI}" effort="1000000" velocity="1" />
+    <limit lower="${-PI}" upper="${PI}" effort="1000000" velocity="3" />
     <dynamics damping="0.7"/>
   </joint>

Commit message: add world

File: tracked_description/urdf/gazebo/tracked_arm_revolute_position.xacro (robot description, xacro)
@@ -97,4 +97,33 @@
     </inertial>
   </link>
+  <joint name="tip_fixed" type="fixed">
+    <parent link="link3"/>
+    <child link="tip_cylinder"/>
+    <origin xyz="0 0 ${height2}" rpy="0 0 0"/>
+  </joint>
+  <!-- Top Link -->
+  <link name="tip_cylinder">
+    <collision>
+      <origin xyz="0 0 0" rpy="0 ${PI/2} ${PI/2}"/>
+      <geometry>
+	<cylinder radius="${width/2}" length="${width}"/>
+      </geometry>
+    </collision>
+    <visual>
+      <origin xyz="0 0 0" rpy="0 ${PI/2} ${PI/2}"/>
+      <geometry>
+	<cylinder radius="${width/2}" length="${width}"/>
+      </geometry>
+      <material name="grey"/>
+    </visual>
+    <inertial>
+      <origin xyz="0 0 0" rpy="0 0 0"/>
+      <mass value="0.000001"/>
+      <inertia
+	  ixx="0.00000001" ixy="0.0" ixz="0.0"
+	  iyy="0.00000001" iyz="0.0"
+	  izz="0.00000001"/>
+    </inertial>
+  </link>
   <joint name="link3_2camera2" type="fixed">
     <parent link="link3"/>

File: tracked_description/urdf/rviz/tracked_arm_continuous_position_rviz.xacro (robot description, xacro)
@@ -97,4 +97,33 @@
     </inertial>
   </link>
+  <joint name="tip_fixed" type="fixed">
+    <parent link="link3"/>
+    <child link="tip_cylinder"/>
+    <origin xyz="0 0 ${height2}" rpy="0 0 0"/>
+  </joint>
+  <!-- Top Link -->
+  <link name="tip_cylinder">
+    <collision>
+      <origin xyz="0 0 0" rpy="0 ${PI/2} ${PI/2}"/>
+      <geometry>
+	<cylinder radius="${width/2}" length="${width}"/>
+      </geometry>
+    </collision>
+    <visual>
+      <origin xyz="0 0 0" rpy="0 ${PI/2} ${PI/2}"/>
+      <geometry>
+	<cylinder radius="${width/2}" length="${width}"/>
+      </geometry>
+      <material name="grey"/>
+    </visual>
+    <inertial>
+      <origin xyz="0 0 0" rpy="0 0 0"/>
+      <mass value="0.000001"/>
+      <inertia
+	  ixx="0.00000001" ixy="0.0" ixz="0.0"
+	  iyy="0.00000001" iyz="0.0"
+	  izz="0.00000001"/>
+    </inertial>
+  </link>
   <joint name="link3_2camera2" type="fixed">
     <parent link="link3"/>
