Commit message: add xacro for real robot and model for test torque sensor

File: tracked_description/urdf/rviz/tracked_arm_continuous_position_rviz_wrs.xacro (robot description, xacro)
@@ -1,11 +1,11 @@
 <?xml version="1.0"?>
 <!-- Revolute-Revolute Manipulator -->
-<robot name="tracked" xmlns:xacro="http://www.ros.org/wiki/xacro">
-  <joint name="base2m1" type="revolute">
-    <parent link="base"/>
+<robot name="tracked_rviz" xmlns:xacro="http://www.ros.org/wiki/xacro">
+  <joint name="box2m1" type="continuous">
+    <parent link="box"/>
     <child link="m1"/>
-    <origin xyz="0 0 ${l_bh/2}" rpy="0 0 ${PI}"/>
+    <origin xyz="0 0 ${0.055}" rpy="0 0 ${PI}"/>
     <axis xyz="0 0 1"/>
-    <limit lower="${-PI}" upper="${PI}" effort="10" velocity="3" />
+<!--    <limit lower="${-PI}" upper="${PI}" effort="1" velocity="1" />-->
     <dynamics damping="0.7"/>
   </joint>
@@ -33,10 +33,10 @@
     </inertial>
   </link>
-  <joint name="joint1" type="revolute">
+  <joint name="joint1" type="continuous">
     <parent link="m1"/>
     <child link="link2"/>
     <origin xyz="0 0 ${m_h}" rpy="0 0 0"/>
     <axis xyz="0 -1 0"/>
-    <limit lower="${-PI}" upper="${PI}" effort="1000000" velocity="3" />
+<!--    <limit lower="${-PI}" upper="${PI}" effort="1" velocity="1" />-->
     <dynamics damping="0.7"/>
   </joint>
@@ -65,10 +65,10 @@
     </inertial>
   </link>
-  <joint name="joint2" type="revolute">
+  <joint name="joint2" type="continuous">
     <parent link="link2"/>
     <child link="link3"/>
     <origin xyz="0 0 ${height2}" rpy="0 0 0"/>
     <axis xyz="0 -1 0"/>
-    <limit lower="${-PI}" upper="${PI}" effort="1000000" velocity="3" />
+<!--    <limit lower="${-PI}" upper="${PI}" effort="1" velocity="1" />-->
     <dynamics damping="0.7"/>
   </joint>
@@ -90,5 +90,5 @@
     <inertial>
       <origin xyz="0 0 ${height3/2}" rpy="0 0 0"/>
-      <mass value="${mass}"/>
+      <mass value="${0.3}"/>
       <inertia
 	  ixx="${mass / 12.0 * (width*width + height3*height3)}" ixy="0.0" ixz="0.0"
@@ -97,12 +97,4 @@
     </inertial>
   </link>
-<!--  <joint name="tip_fixed" type="continuous">-->
-<!--    <parent link="link3"/>-->
-<!--    <child link="tip_cylinder"/>-->
-<!--    <origin xyz="0 0 ${height2}" rpy="0 0 0"/>-->
-<!--    <axis xyz="0 -1 0"/>-->
-<!--    <limit lower="${-PI}" upper="${PI}" effort="10000000000000" velocity="3" />-->
-<!--    <dynamics damping="0.7"/>-->
-<!--  </joint>-->
   <joint name="tip_fixed" type="fixed">
     <parent link="link3"/>
@@ -127,5 +119,5 @@
     <inertial>
       <origin xyz="0 0 0" rpy="0 0 0"/>
-      <mass value="0.00001"/>
+      <mass value="0.000001"/>
       <inertia
 	  ixx="0.00000001" ixy="0.0" ixz="0.0"
@@ -183,4 +175,28 @@
   <link name="camera2_optical">
   </link>
+  <link name="m1_origin"/>
+  <joint name="m1_2link2_origin" type="fixed">
+    <parent link="m1"/>
+    <child link="m1_origin"/>
+    <origin xyz="0 0 ${m_h/2}" rpy="0 0 0"/>
+  </joint>
+  <link name="link2_origin"/>
+  <joint name="link2_2link2_origin" type="fixed">
+    <parent link="link2"/>
+    <child link="link2_origin"/>
+    <origin xyz="0 0 ${height2/2}" rpy="0 0 0"/>
+  </joint>
+  <link name="link3_origin"/>
+  <joint name="link3_2link3_origin" type="fixed">
+    <parent link="link3"/>
+    <child link="link3_origin"/>
+    <origin xyz="0 0 ${height2/2}" rpy="0 0 0"/>
+  </joint>
+  <link name="link3_tip"/>
+  <joint name="link3_2link3_tip" type="fixed">
+    <parent link="link3"/>
+    <child link="link3_tip"/>
+    <origin xyz="0 0 ${height2}" rpy="0 0 0"/>
+  </joint>
   <transmission name="tran_base2m1">
     <type>transmission_interface/SimpleTransmission</type>
@@ -213,44 +229,3 @@
     </actuator>
   </transmission>
-<!--  <transmission name="tran_tip_fixed">-->
-<!--    <type>transmission_interface/SimpleTransmission</type>-->
-<!--    <joint name="tip_fixed">-->
-<!--      <hardwareInterface>PositionJointInterface</hardwareInterface>-->
-<!--    </joint>-->
-<!--    <actuator name="motor_tip_fixed">-->
-<!--      <hardwareInterface>PositionJointInterface</hardwareInterface>-->
-<!--      <mechanicalReduction>1</mechanicalReduction>-->
-<!--    </actuator>-->
-<!--  </transmission>-->
-<!-- Force and torque sensor -->
-  <gazebo reference="joint1">
-    <provideFeedback>true</provideFeedback>
-  </gazebo>
-  <gazebo>
-    <plugin name="ft_sensor" filename="libgazebo_ros_ft_sensor.so">
-      <updateRate>100.0</updateRate>
-      <topicName>/tracked/ft_sensor_joint1</topicName>
-      <jointName>joint1</jointName>
-    </plugin>
-  </gazebo>
-  <gazebo reference="joint2">
-    <provideFeedback>true</provideFeedback>
-  </gazebo>
-  <gazebo>
-    <plugin name="ft_sensor" filename="libgazebo_ros_ft_sensor.so">
-      <updateRate>100.0</updateRate>
-      <topicName>/tracked/ft_sensor_joint2</topicName>
-      <jointName>joint2</jointName>
-    </plugin>
-  </gazebo>
-  <gazebo reference="tip_fixed">
-    <provideFeedback>true</provideFeedback>
-  </gazebo>
-  <gazebo>
-    <plugin name="ft_sensor" filename="libgazebo_ros_ft_sensor.so">
-      <updateRate>100.0</updateRate>
-      <topicName>/tracked/ft_sensor_tip_fixed</topicName>
-      <jointName>tip_fixed</jointName>
-    </plugin>
-  </gazebo>
 </robot>

File: tracked_description/urdf/rviz/tracked_rviz_wrs.xacro (robot description, xacro)
@@ -1,8 +1,8 @@
 <?xml version="1.0"?>
 <!-- Revolute-Revolute Manipulator -->
-<robot name="tracked" xmlns:xacro="http://www.ros.org/wiki/xacro">
+<robot name="tracked_rviz" xmlns:xacro="http://www.ros.org/wiki/xacro">
   <!-- Constants for robot dimensions -->
   <xacro:property name="PI" value="3.1415926535897931"/>
-  <xacro:property name="m_f" value="200" /> <!-- flipper mass -->
+  <xacro:property name="m_f" value="1" /> <!-- flipper mass -->
   <xacro:property name="m_b" value="30" /> <!-- main mass -->
   <xacro:property name="m_1" value="0.2" /> <!-- motor1 mass -->
@@ -21,7 +21,7 @@
   <xacro:property name="l_ba" value="0.20" /> <!-- main axis width -->
   <xacro:property name="l_1" value="1" /> <!-- l1 -->
-  <xacro:property name="l_2" value="0.30" /> <!-- link2 length -->
-  <xacro:property name="l_3" value="0.30" /> <!-- link3 length -->
-  <xacro:property name="m_h" value="0.05" /> <!-- motor height -->
+  <xacro:property name="l_2" value="0.2215" /> <!-- link2 length -->
+  <xacro:property name="l_3" value="0.232" /> <!-- link3 length -->
+  <xacro:property name="m_h" value="0.105" /> <!-- motor height -->
   <xacro:property name="width" value="0.05" /> <!-- Square dimensions (widthxwidth) of beams -->
   <xacro:property name="height1" value="2" /> <!-- Link 1 -->
@@ -36,21 +36,37 @@
   <xacro:property name="axel_offset" value="0.05" /> <!-- Space btw top of beam and the each joint -->
   <!-- Import all Gazebo-customization elements, including Gazebo colors -->
-  <xacro:include filename="$(find tracked_description)/urdf/gazebo/tracked.gazebo" />
+<!--  <xacro:include filename="$(find tracked_description)/urdf/rviz/tracked_rviz.gazebo" />-->
   <!-- Import Rviz colors -->
-  <xacro:include filename="$(find tracked_description)/urdf/gazebo/materials.xacro" />
+  <xacro:include filename="$(find tracked_description)/urdf/rviz/materials_wrs.xacro" />
 <!-- arm xacro files-->
 <!--You can import one of them-->
-<!--  <xacro:include filename="$(find tracked_description)/urdf/gazebo/tracked_arm_continuous_position.xacro" />-->
-  <xacro:include filename="$(find tracked_description)/urdf/gazebo/tracked_arm_revolute_position.xacro" />
-<!--  <xacro:include filename="$(find tracked_description)/urdf/gazebo/tracked_arm_revolute_effort.xacro" />-->
-<!-- fake crawler xacro files-->
-<!-- This model is not completed-->
-<!--  <xacro:include filename="$(find tracked_description)/urdf/gazebo/tracked_wheel.xacro" />-->
+<!--  <xacro:include filename="$(find tracked_description)/urdf/rviz/tracked_arm_revolute_position.xacro" />-->
+<!--  <xacro:include filename="$(find tracked_description)/urdf/rviz/tracked_arm_revolute_effort.xacro" />-->
   <!-- Used for fixing robot to Gazebo 'base_link' -->
-  <link name="world"/>
-  <joint name="world2base" type="floating">
-    <parent link="world"/>
-    <child link="base"/>
-  </joint>
+	<link name="world"/>
+	<joint name="world2xbase" type="floating">
+		<parent link="world"/>
+		<child link="xbase"/>
+	</joint>
+	<link name="xbase">
+		<origin xyz="0 0 0" rpy="0 0 0"/>
+	</link>
+	<joint name="xbase_ybase" type="continuous">
+		<parent link="xbase"/>
+		<child link="ybase"/>
+		<origin rpy="0 0 0" xyz="0 0 0"/>
+		<axis xyz="1 0 0"/>
+<!--		<limit effort="20" lower="-2.0" upper="2.0" velocity="1"/>-->
+	</joint>
+	<link name="ybase">
+		<origin xyz="0 0 0" rpy="0 0 0"/>
+	</link>
+	<joint name="ybase_base" type="continuous">
+		<parent link="ybase"/>
+		<child link="base"/>
+		<origin rpy="0 0 0" xyz="0 0 0"/>
+		<axis xyz="0 1 0"/>
+<!--		<limit effort="20" lower="-2.0" upper="2.0" velocity="1"/>-->
+	</joint>
   <!-- Base Link -->
   <link name="base">
@@ -77,10 +93,29 @@
     </inertial>
   </link>
-  <joint name="base2FL" type="revolute">
+  <link name="robot_origin"/>
+  <joint name="base2robot_origin" type="fixed">
+    <parent link="base"/>
+    <child link="robot_origin"/>
+    <origin xyz="0 0 ${-l_bh/2}" rpy="0 0 0"/>
+  </joint>
+  <joint name="base2box" type="fixed">
+    <parent link="base"/>
+    <child link="box"/>
+    <origin xyz="0 0 ${l_bh/2+0.055}" rpy="0 0 0"/>
+  </joint>
+  <link name="box">
+    <visual>
+      <origin xyz="0 0 0" rpy="0 0 0"/>
+      <geometry>
+	<box size="0.4 0.23 0.11"/>
+      </geometry>
+      <material name="grey"/>
+    </visual>
+  </link>
+  <joint name="base2FL" type="continuous">
     <parent link="base"/>
     <child link="FL"/>
-    <origin xyz="${l_ba/2} ${l_bw/2 + l_fw/2} 0" rpy="0 0 0"/>
+    <origin xyz="${l_ba/2} ${l_bw/2 + l_fw/2 + 0.01} 0" rpy="0 0 0"/>
     <axis xyz="0 1 0"/>
-    <limit lower="${-PI}" upper="${PI}" effort="1000000" velocity="3" />
     <dynamics damping="0.7"/>
   </joint>
@@ -108,10 +143,9 @@
     </inertial>
   </link>
-  <joint name="base2RL" type="revolute">
+  <joint name="base2RL" type="continuous">
     <parent link="base"/>
     <child link="RL"/>
-    <origin xyz="${-l_ba/2} ${l_bw/2 + l_fw/2} 0" rpy="0 0 0"/>
+    <origin xyz="${-l_ba/2} ${l_bw/2 + l_fw/2 + 0.01} 0" rpy="0 0 0"/>
     <axis xyz="0 1 0"/>
-    <limit lower="${-PI}" upper="${PI}" effort="1000000" velocity="3" />
     <dynamics damping="0.7"/>
   </joint>
@@ -139,10 +173,9 @@
     </inertial>
   </link>
-  <joint name="base2FR" type="revolute">
+  <joint name="base2FR" type="continuous">
     <parent link="base"/>
     <child link="FR"/>
-    <origin xyz="${l_ba/2} ${-(l_bw/2 + l_fw/2)} 0" rpy="0 0 0"/>
+    <origin xyz="${l_ba/2} ${-(l_bw/2 + l_fw/2 + 0.01)} 0" rpy="0 0 0"/>
     <axis xyz="0 1 0"/>
-    <limit lower="${-PI}" upper="${PI}" effort="1000000" velocity="3" />
     <dynamics damping="0.7"/>
   </joint>
@@ -170,10 +203,9 @@
     </inertial>
   </link>
-  <joint name="base2RR" type="revolute">
+  <joint name="base2RR" type="continuous">
     <parent link="base"/>
     <child link="RR"/>
-    <origin xyz="${-l_ba/2} ${-(l_bw/2 + l_fw/2)} 0" rpy="0 0 0"/>
+    <origin xyz="${-l_ba/2} ${-(l_bw/2 + l_fw/2 + 0.01)} 0" rpy="0 0 0"/>
     <axis xyz="0 1 0"/>
-    <limit lower="${-PI}" upper="${PI}" effort="1000000" velocity="3" />
     <dynamics damping="0.7"/>
   </joint>
@@ -203,5 +235,5 @@
   <joint name="base2hokuyo" type="fixed">
     <axis xyz="0 1 0" />
-    <origin xyz="${l_ba/3+0.02} 0 ${l_bh/2+0.03}" rpy="0 0 0"/>
+    <origin xyz="${l_ba/3+0.1} 0 ${l_bh/2+0.03+0.11}" rpy="0 0 0"/>
     <parent link="base"/>
     <child link="hokuyo"/>
@@ -216,43 +248,64 @@
     </visual>
   </link>
-  <transmission name="tran_base2FL">
-    <type>transmission_interface/SimpleTransmission</type>
-    <joint name="base2FL">
-      <hardwareInterface>PositionJointInterface</hardwareInterface>
-    </joint>
-    <actuator name="motor_base2FL">
-      <hardwareInterface>PositionJointInterface</hardwareInterface>
-      <mechanicalReduction>1</mechanicalReduction>
-    </actuator>
-  </transmission>
-  <transmission name="tran_base2RL">
-    <type>transmission_interface/SimpleTransmission</type>
-    <joint name="base2RL">
-      <hardwareInterface>PositionJointInterface</hardwareInterface>
-    </joint>
-    <actuator name="motor_base2RL">
-      <hardwareInterface>PositionJointInterface</hardwareInterface>
-      <mechanicalReduction>1</mechanicalReduction>
-    </actuator>
-  </transmission>
-  <transmission name="tran_base2FR">
-    <type>transmission_interface/SimpleTransmission</type>
-    <joint name="base2FR">
-      <hardwareInterface>PositionJointInterface</hardwareInterface>
-    </joint>
-    <actuator name="motor_base2FR">
-      <hardwareInterface>PositionJointInterface</hardwareInterface>
-      <mechanicalReduction>1</mechanicalReduction>
-    </actuator>
-  </transmission>
-  <transmission name="tran_base2RR">
-    <type>transmission_interface/SimpleTransmission</type>
-    <joint name="base2RR">
-      <hardwareInterface>PositionJointInterface</hardwareInterface>
-    </joint>
-    <actuator name="motor_base2RR">
-      <hardwareInterface>PositionJointInterface</hardwareInterface>
-      <mechanicalReduction>1</mechanicalReduction>
-    </actuator>
-  </transmission>
+  <link name="FL_origin"/>
+  <joint name="FL2FL_origin" type="fixed">
+    <parent link="FL"/>
+    <child link="FL_origin"/>
+    <origin xyz="${l_fa/2} 0 0" rpy="0 0 0"/>
+  </joint>
+  <link name="FR_origin"/>
+  <joint name="FR2FR_origin" type="fixed">
+    <parent link="FR"/>
+    <child link="FR_origin"/>
+    <origin xyz="${l_fa/2} 0 0" rpy="0 0 0"/>
+  </joint>
+  <link name="RL_origin"/>
+  <joint name="RL2RL_origin" type="fixed">
+    <parent link="RL"/>
+    <child link="RL_origin"/>
+    <origin xyz="${-l_fa/2} 0 0" rpy="0 0 0"/>
+  </joint>
+  <link name="RR_origin"/>
+  <joint name="RR2RR_origin" type="fixed">
+    <parent link="RR"/>
+    <child link="RR_origin"/>
+    <origin xyz="${-l_fa/2} 0 0" rpy="0 0 0"/>
+  </joint>
+  <link name="FL_tip"/>
+  <joint name="FL2FL_tip" type="fixed">
+    <parent link="FL"/>
+    <child link="FL_tip"/>
+    <origin xyz="${l_fa} 0 0" rpy="0 0 0"/>
+  </joint>
+  <link name="FR_tip"/>
+  <joint name="FR2FR_tip" type="fixed">
+    <parent link="FR"/>
+    <child link="FR_tip"/>
+    <origin xyz="${l_fa} 0 0" rpy="0 0 0"/>
+  </joint>
+  <link name="RL_tip"/>
+  <joint name="RL2RL_tip" type="fixed">
+    <parent link="RL"/>
+    <child link="RL_tip"/>
+    <origin xyz="${-l_fa} 0 0" rpy="0 0 0"/>
+  </joint>
+  <link name="RR_tip"/>
+  <joint name="RR2RR_tip" type="fixed">
+    <parent link="RR"/>
+    <child link="RR_tip"/>
+    <origin xyz="${-l_fa} 0 0" rpy="0 0 0"/>
+  </joint>
+  <link name="right_rollover_axis"/>
+  <joint name="robot_origin2right_rollover_axis" type="fixed">
+    <parent link="robot_origin"/>
+    <child link="right_rollover_axis"/>
+    <origin xyz="0 ${-l_bw/2-l_fw} 0" rpy="0 0 0"/>
+  </joint>
+  <link name="left_rollover_axis"/>
+  <joint name="robot_origin2left_rollover_axis" type="fixed">
+    <parent link="robot_origin"/>
+    <child link="left_rollover_axis"/>
+    <origin xyz="0 ${l_bw/2+l_fw} 0" rpy="0 0 0"/>
+  </joint>
+  <xacro:include filename="$(find tracked_description)/urdf/rviz/tracked_arm_continuous_position_rviz_wrs.xacro" />
 </robot>
